File: Test2.kicad_pcb (KiCad board)
At the start: 2 copper layers, 82 x 61 mm, 19 parts, among them J1 Raspberry_Pi_2_3, J1_GPIO4 01×06, J2_GPIO17 Conn_01x06_Socket, J3_GPIO27 Conn_01x06_Socket, J4_GPIO22 Conn_01x06_Socket, M1_GPIO23 Motor_Servo, SW1_GPIO8 SW_Push

Commit message: Initial commit
Parts:
- added J2: Conn_01x04_Pin, Library:Grove_1x04, F.Cu at (156.0, 124.5)
- added R3: 100Ω, Resistor_SMD:R_0805_2012Metric, F.Cu at (125.5, 102.1)
- added R4: 100Ω, Resistor_SMD:R_0805_2012Metric, F.Cu at (132.5, 88.4)
- added R5: 100Ω, Resistor_SMD:R_0805_2012Metric, F.Cu at (132.5, 92.6)
Connections:
- Fan1 pad 1: Net-(Fan1-Pin_1) -> Net-(D1-K)
- J1 pad 10: unconnected-(J1-GPIO15/RXD-Pad10) -> Net-(J1-GPIO15/RXD)
- J1 pad 14: Net-(Fan1-Pin_1) -> Net-(D1-K)
- J1 pad 18: Net-(D2-A) -> Net-(J1-GPIO24)
- J1 pad 20: Net-(Fan1-Pin_1) -> Net-(D1-K)
- J1 pad 22: Net-(D3-A) -> Net-(J1-GPIO25)
- J1 pad 25: Net-(Fan1-Pin_1) -> Net-(D1-K)
- J1 pad 26: Net-(D1-A) -> Net-(J1-~{CE1}/GPIO7)
- J1 pad 30: Net-(Fan1-Pin_1) -> Net-(D1-K)
- J1 pad 34: Net-(Fan1-Pin_1) -> Net-(D1-K)
- J1 pad 37: Net-(D4-A) -> Net-(J1-GPIO26)
- J1 pad 39: Net-(Fan1-Pin_1) -> Net-(D1-K)
- J1 pad 6: Net-(Fan1-Pin_1) -> Net-(D1-K)
- J1 pad 8: unconnected-(J1-GPIO14/TXD-Pad8) -> Net-(J1-GPIO14/TXD)
- J1 pad 9: Net-(Fan1-Pin_1) -> Net-(D1-K)
- M1_GPIO23 pad 3: Net-(Fan1-Pin_1) -> Net-(D1-K)
- R1 pad 1: Net-(R1-Pad1) -> Net-(J1-3V3-Pad1)
- R1 pad 2: Net-(J1-~{CE0}/GPIO8) -> Net-(R1-Pad2)
- R2 pad 1: Net-(D1-K) -> Net-(D1-A)
- R2 pad 2: Net-(Fan1-Pin_1) -> Net-(J1-~{CE1}/GPIO7)
